File: hardware/sheet4.kicad_sch (KiCad schematic)
At the start: 27 parts, among them J2 B4B-XH-A, J3 B-2100S04P-A110, J4 U254-051N-4BH806, U2 STM32F072CBT6, U4 USBLC6-2SC6, Y1 32.768kHz

Commit message: hardware(feat): update stm32 pinout
Parts:
- added TP1: 1.0P-SMD, 12_mechanical:TestPoint_Pad_D1.0mm, symbol 12_mechanical:TP_1.0P-SMD
Connections:
- net MCO: now reaches U2.29 (PA8)
- net MCO: now also TP1.1
- no-connect marks 1 -> 14
Changed lines of the file:
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@@
 	)
 	(no_connect
+		(at 185.42 127)
+	)
+	(no_connect
+		(at 185.42 106.68)
+	)
+	(no_connect
+		(at 185.42 83.82)
+	)
+	(no_connect
+		(at 185.42 139.7)
+	)
+	(no_connect
+		(at 185.42 124.46)
+	)
+	(no_connect
+		(at 139.7 114.3)
+	)
+	(no_connect
+		(at 185.42 137.16)
+	)
+	(no_connect
 		(at 264.16 88.9)
 	)
+	(no_connect
+		(at 139.7 121.92)
+	)
+	(no_connect
+		(at 185.42 129.54)
+	)
+	(no_connect
+		(at 185.42 119.38)
+	)
+	(no_connect
+		(at 139.7 116.84)
+	)
+	(no_connect
+		(at 185.42 81.28)
+	)
+	(no_connect
+		(at 185.42 86.36)
+	)
 	(wire
 		(pts
@@
 	(wire
 		(pts
+			(xy 185.42 93.98) (xy 198.12 93.98)
+		)
+		(stroke
+			(width 0)
+			(type default)
+		)
+	)
+	(wire
+		(pts
 			(xy 256.54 86.36) (xy 264.16 86.36)
 		)
@@
 		)
 	)
+	(label "MCO"
+		(at 198.12 93.98 180)
+		(effects
+			(font
+				(size 1.27 1.27)
+			)
+			(justify right bottom)
+		)
+	)
 	(label "SWDIO"
 		(at 66.04 114.3 180)
@@
 		)
 		(pin "4"
-			(alternate "RCC_OSC32_OUT (PC15)")
+			(alternate "PC15/RCC_OSC32_OUT")
 		)
 		(pin "8"
@@
 		)
 		(pin "28"
-			(alternate "SPI2_MOSI (PB15)")
+			(alternate "PB15/SPI2_MOSI")
 		)
 		(pin "35"
@@
 		)
 		(pin "31"
-			(alternate "USART1_RX (PA10)")
+			(alternate "PA10/USART1_RX")
 		)
 		(pin "48"
@@
 		)
 		(pin "22"
-			(alternate "USART3_RX (PB11)")
+			(alternate "PB11/USART3_RX")
 		)
 		(pin "45"
 		)
 		(pin "21"
-			(alternate "USART3_TX (PB10)")
+			(alternate "PB10/USART3_TX")
 		)
 		(pin "25"
@@
 		)
 		(pin "27"
-			(alternate "SPI2_MISO (PB14)")
+			(alternate "PB14/SPI2_MISO")
 		)
 		(pin "13"
@@
 		)
 		(pin "3"
-			(alternate "RCC_OSC32_IN (PC14)")
+			(alternate "PC14/RCC_OSC32_IN")
 		)
 		(pin "1"
 		)
 		(pin "26"
-			(alternate "SPI2_SCK (PB13)")
+			(alternate "PB13/SPI2_SCK")
 		)
 		(pin "11"
@@
 		)
 		(pin "29"
+			(alternate "PA8/RCC_MCO")
 		)
 		(pin "30"
-			(alternate "USART1_TX (PA9)")
+			(alternate "PA9/USART1_TX")
 		)
 		(pin "10"
@@
 		)
 		(pin "32"
-			(alternate "USB_DM (PA11)")
+			(alternate "PA11/USB_DM")
 		)
 		(pin "18"
 		)
 		(pin "42"
-			(alternate "I2C1_SCL (PB6)")
+			(alternate "PB6/USART1_TX")
 		)
 		(pin "40"
 		)
 		(pin "33"
-			(alternate "USB_DP (PA12)")
+			(alternate "PA12/USB_DP")
 		)
 		(pin "19"
 		)
 		(pin "43"
-			(alternate "I2C1_SDA (PB7)")
+			(alternate "PB7/I2C1_SDA")
 		)
 		(pin "34"
-			(alternate "SWDIO (PA13)")
+			(alternate "SWDIO")
 		)
 		(pin "38"
 		)
 		(pin "37"
-			(alternate "SWCLK (PA14)")
+			(alternate "SWCLK")
 		)
 		(pin "41"
@@
 					(unit 1)
 				)
+			)
+		)
+	)
+	(symbol
+		(lib_id "12_mechanical:TP_1.0P-SMD")
+		(at 203.2 93.98 270)
+		(unit 1)
+		(exclude_from_sim no)
+		(in_bom no)
+		(on_board yes)
+		(dnp no)
+		(property "Reference" "TP1"
+			(at 203.835 93.98 90)
+			(effects
+				(font
+					(size 1.27 1.27)
+				)
+				(justify left)
+			)
+		)
+		(property "Value" "1.0P-SMD"
+			(at 204.47 95.25 90)
+			(effects
+				(font
+					(size 1.27 1.27)
+				)
+				(justify left)
+				(hide yes)
+			)
+		)
+		(property "Footprint" "12_mechanical:TestPoint_Pad_D1.0mm"
+			(at 203.2 93.98 0)
+			(effects
+				(font
+					(size 1.27 1.27)
+				)
+				(hide yes)
+			)
+		)
+		(property "Datasheet" ""
+			(at 203.2 93.98 0)
+			(effects
+				(font
+					(size 1.27 1.27)
+				)
+				(hide yes)
+			)
+		)
+		(property "Description" "TEST POINT 1.0mm SMD PAD probe or bed of nails board feature not a purchased part"
+			(at 203.2 93.98 0)
+			(effects
+				(font
+					(size 1.27 1.27)
+				)
+				(hide yes)
+			)
+		)
+		(property "Package" "SMD"
+			(at 203.2 93.98 0)
+			(effects
+				(font
+					(size 1.27 1.27)
+				)
+				(hide yes)
+			)
+		)
+		(pin "1"
+		)
+		(instances
+			(project ""
+				(path "/08767502-fa14-4976-aaca-9650785a2144/90f70198-c0ab-4cef-90bd-cd1364d30a2f"
+					(reference "TP1")
+					(unit 1)
+				)
