File: hardware/sheet3.kicad_sch (KiCad schematic)
At the start: 31 parts, among them J1 DC-005-5A-2.0, U1 AP63205WU-7, U3 AP2114H-3.3TRG1

Commit message: hardware(feat): complete pcb placement, closes #15
Parts:
- removed FID1, FID2, FID3, FID4: 1.0P-2.0M, 12_mechanical:Fiducial_1mm_Mask2mm, symbol 12_mechanical:FID_1.0P-2.0M
