File: hardware/chronolog.kicad_pcb (KiCad board)
At the start: 4 copper layers, 100 x 50 mm, 95 parts, among them J1 DC-005-5A-2.0, J2 B4B-XH-A, J3 B-2100S04P-A110, J4 U254-051N-4BH806, Q1 BSS138, Q2 BSS138, Q3 BC817-40LT1G, U1 AP63205WU-7, U2 STM32F072CBT6, U3 AP2114H-3.3TRG1, U4 USBLC6-2SC6, U5 W25Q32JVSNIQ, U6 LM75BD, U7 ESP-01, U8 WC1602A, U9 PCF8574T, Y1 32.768kHz

Commit message: hardware(feat): complete pcb routing, closes #16
Routing:
- net GND: vias 61 -> 248

Commit message: hardware(feat): review the board, closes #17
Other:
- board text added: "BUTTONS + LED RGB"
- board text added: "LCD"
- board text added: "MCU"
- board text added: "NOR + TEMP SENSOR"
- board text added: "RTC BATTERY"
- board text removed: "MCU STM32 + NOR FLASH"
- board text removed: "RTC BATTERY (BT1)"
- board text removed: "TEMP (LM75) + SWD/UART"
- board text removed: "USB IN"
- board text removed: "[BOTTOM] BUTTONS + RGB LED"
- board text removed: "[BOTTOM] LCD 16x2 (WC1602A)"
