File: hardware/chronolog.kicad_sch (KiCad schematic)
At the start: 0 parts

Commit message: hardware(feat): add lcd sheet
Other:
- added sheet [08] - LCD (sheet8.kicad_sch)
- note added: "LCD"
Changed lines of the file:
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@@
 		)
 	)
-	(text "..........................................."
+	(text "LCD"
 		(exclude_from_sim no)
 		(at 44.45 133.35 0)
@@
 				)
 			)
+		)
+	)
+	(sheet
+		(at 353.06 318.77)
+		(size 29.21 3.81)
+		(exclude_from_sim no)
+		(in_bom yes)
+		(on_board yes)
+		(dnp no)
+		(fields_autoplaced yes)
+		(stroke
+			(width 0.1524)
+			(type solid)
+		)
+		(fill
+			(color 0 0 0 0.0000)
+		)
+		(property "Sheetname" "[08] - LCD"
+			(at 353.06 318.0584 0)
+			(effects
+				(font
+					(size 1.27 1.27)
+				)
+				(justify left bottom)
+			)
+		)
+		(property "Sheetfile" "sheet8.kicad_sch"
+			(at 353.06 323.1646 0)
+			(effects
+				(font
+					(size 1.27 1.27)
+				)
+				(justify left top)
+			)
+		)
+		(instances
+			(project "chronolog"
+				(path "/08767502-fa14-4976-aaca-9650785a2144"
+					(page "8")
+				)
+			)

Commit message: hardware(feat): add board layers and assembly drawing sheets
Other:
- added sheet [09] - Board Layers (sheet9.kicad_sch)
- added sheet [10] - Assembly Drawing (sheet10.kicad_sch)
- note added: "Assembly Drawing"
- note added: "Board Layers"
Changed lines of the file:
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@@
 		)
 	)
-	(text "..........................................."
+	(text "Board Layers"
 		(exclude_from_sim no)
 		(at 44.45 140.97 0)
@@
 		)
 	)
-	(text "..........................................."
+	(text "Assembly Drawing"
 		(exclude_from_sim no)
 		(at 44.45 148.59 0)
@@
 				)
 			)
+		)
+	)
+	(sheet
+		(at 287.02 330.2)
+		(size 29.21 3.81)
+		(exclude_from_sim no)
+		(in_bom yes)
+		(on_board yes)
+		(dnp no)
+		(fields_autoplaced yes)
+		(stroke
+			(width 0.1524)
+			(type solid)
+		)
+		(fill
+			(color 0 0 0 0.0000)
+		)
+		(property "Sheetname" "[10] - Assembly Drawing"
+			(at 287.02 329.4884 0)
+			(effects
+				(font
+					(size 1.27 1.27)
+				)
+				(justify left bottom)
+			)
+		)
+		(property "Sheetfile" "sheet10.kicad_sch"
+			(at 287.02 334.5946 0)
+			(effects
+				(font
+					(size 1.27 1.27)
+				)
+				(justify left top)
+			)
+		)
+		(instances
+			(project "chronolog"
+				(path "/08767502-fa14-4976-aaca-9650785a2144"
+					(page "10")
+				)
+			)
+		)
+	)
+	(sheet
+		(at 386.08 318.77)
+		(size 29.21 3.81)
+		(exclude_from_sim no)
+		(in_bom yes)
+		(on_board yes)
+		(dnp no)
+		(fields_autoplaced yes)
+		(stroke
+			(width 0.1524)
+			(type solid)
+		)
+		(fill
+			(color 0 0 0 0.0000)
+		)
+		(property "Sheetname" "[09] - Board Layers"
+			(at 386.08 318.0584 0)
+			(effects
+				(font
+					(size 1.27 1.27)
+				)
+				(justify left bottom)
+			)
+		)
+		(property "Sheetfile" "sheet9.kicad_sch"
+			(at 386.08 323.1646 0)
+			(effects
+				(font
+					(size 1.27 1.27)
+				)
+				(justify left top)
+			)
+		)
+		(instances
+			(project "chronolog"
+				(path "/08767502-fa14-4976-aaca-9650785a2144"
+					(page "9")
+				)
+			)
